Commit message: Add files via upload

File: src/bot1/urdf/bot1_updated.urdf (robot description, URDF)
Before this commit: robot bot1, 14 links, 13 joints
Links:
- added link sonar_link, mass 1e-5; collision box size=0.01 0.01 0.01; visual box size=0.01 0.01 0.01
- link FLW: mass 0.16694 -> 0.23606; geometry collision mesh filename=package://bot4/meshes/FLW.STL; visual mesh filename=package://bot4/meshes/FLW.STL
- link FRW: mass 0.16694 -> 0.23606; geometry collision mesh filename=package://bot4/meshes/FRW.STL; visual mesh filename=package://bot4/meshes/FRW.STL
- link LA: mass 0.11493 -> 0.069926; geometry collision mesh filename=package://bot4/meshes/LA.STL; visual mesh filename=package://bot4/meshes/LA.STL
- link LF: geometry collision mesh filename=package://bot4/meshes/LF.STL; visual mesh filename=package://bot4/meshes/LF.STL
- link RA: mass 0.11493 -> 0.069926; geometry collision mesh filename=package://bot4/meshes/RA.STL; visual mesh filename=package://bot4/meshes/RA.STL
- link RF: geometry collision mesh filename=package://bot4/meshes/RF.STL; visual mesh filename=package://bot4/meshes/RF.STL
- link RLW: mass 0.16694 -> 0.23606; geometry collision mesh filename=package://bot4/meshes/RLW.STL; visual mesh filename=package://bot4/meshes/RLW.STL
- link RRW: mass 0.16694 -> 0.23606; geometry collision mesh filename=package://bot4/meshes/RRW.STL; visual mesh filename=package://bot4/meshes/RRW.STL
- link base_link: mass 2.0304 -> 2.519; geometry collision mesh filename=package://bot4/meshes/base_link.STL; visual mesh filename=package://bot4/meshes/base_link.STL
Joints:
- added joint sonar_front_joint: type fixed, parent LA, child sonar_link, origin xyz=0.09 0.015 -0.02 rpy=3.1415926 0 -1.570796326, axis 0 1 0
- joint BJ: limit lower=-0.15 upper=0 effort=10 velocity=0.1 -> lower=-0.15 upper=0 effort=1000 velocity=0.1
- joint FJ: limit lower=-0.18 upper=0 effort=10 velocity=0.1 -> lower=-0.18 upper=0 effort=10 velocity=0.05
- joint FLWJ: origin xyz=0.095 0.17 0.047 rpy=1.5707963267949 0 0 -> xyz=0.145 0.17 0.047 rpy=1.5707963267949 0 0
- joint FRWJ: origin xyz=0.095 -0.17 0.047 rpy=1.5707963267949 0.39309481042652 -3.14159265358979 -> xyz=0.145 -0.17 0.047 rpy=1.5707963267949 0.39309481042652 -3.14159265358979
- joint LAJ: origin xyz=0.175 0.185 0.055 rpy=1.5708 0 0 -> xyz=0.175 0.185 0.055 rpy=1.5707963267949 0 0
- joint LFJ: limit lower=-0.34 upper=1.36 effort=100 velocity=0.15 -> lower=-0.9 upper=0.8 effort=100 velocity=0.125; mimic joint=RFJ multiplier=-1 offset=0 -> (none); origin xyz=0.135 0 0 rpy=0 -0.64739 0 -> xyz=0.085 0 0 rpy=0 -0.64739213973993 0
- joint RFJ: limit lower=-1.5 upper=0.2 effort=100 velocity=0.15 -> lower=-0.8 upper=0.9 effort=100 velocity=0.125; origin xyz=0.135 0 0 rpy=0 0.7854 0 -> xyz=0.085 0 0 rpy=0 0.78539816339745 0
- joint RLWJ: origin xyz=-0.065 0.17 0.047 rpy=1.5707963267949 0 0 -> xyz=-0.150 0.17 0.047 rpy=1.5707963267949 0 0
- joint RRWJ: origin xyz=-0.065 -0.17 0.047 rpy=1.5707963267949 0.393094810426521 -3.14159265358979 -> xyz=-0.150 -0.17 0.047 rpy=1.5707963267949 0.393094810426521 -3.14159265358979
- joint hokuyo_joint: origin xyz=0.04 0.05 0 rpy=-1.57 0 0 -> xyz=0.04 0.04 0 rpy=-1.57 0 0
